Commit message: changes to pen and surface positions. add rviz default config.  add path planner and motion controller initial setup

File: urdf/pen.xacro (robot description, xacro)
@@ -36,4 +36,10 @@
             <child link="${name}_link" />
         </joint>
+        <link name="${name}_tip"/>
+        <joint name="${name}_link-tip_joint" type="fixed">
+            <origin xyz="0 0 0.077" rpy="0 0 0"/>
+            <parent link="${name}_link"/>
+            <child link="${name}_tip"/>
+        </joint>
     </xacro:macro>
 </robot>

File: urdf/surface.xacro (robot description, xacro)
@@ -30,5 +30,5 @@
         </link>
         <joint name="${name}_joint" type="fixed">
-            <origin xyz="0.8 0 0" rpy="0 0 0" />
+            <origin xyz="1.5 0 0" rpy="0 0 0" />
             <parent link="world" />
             <child link="${name}_link" />
